Commit message: Update a6x_macro.urdf.xacro too, as we update robot's urdf

File: a6x_description/urdf/a6x_macro.urdf.xacro (robot description, xacro)
@@ -12,21 +12,21 @@
             <visual>
                 <geometry>
-                <mesh filename="package://a6x_description/meshes/visual/base_link.STL" />
-                </geometry>
-                <origin xyz="0.000 0.000 0.000" rpy="0.000 0.000 0.000" />
-                <material name="grey" />
-            </visual>
-            <collision>
-                <geometry>
-                <mesh filename="package://a6x_description/meshes/visual/base_link.STL" />
-                </geometry>
-                <origin xyz="0.000 0.000 0.000" rpy="0.000 0.000 0.000" />
-            </collision>
-            <inertial>
-                <mass value="2.052381" />
-                <origin xyz="0.010773 -0.013141 0.019508" rpy="0 0 0" />
-                <inertia ixx="0.007060" ixy="-0.000705" ixz="-0.000013"
-                        iyy="0.003238" iyz="0.000167"
-                        izz="0.009216" />
+                    <mesh filename="package://a6x_description/meshes/visual/base_link.STL" />
+                </geometry>
+                    <origin xyz="0.000 0.000 0.000" rpy="0.000 0.000 0.000" />
+                <material name="grey" />
+            </visual>
+            <collision>
+                <geometry>
+                    <mesh filename="package://a6x_description/meshes/visual/base_link.STL" />
+                </geometry>
+                <origin xyz="0.000 0.000 0.000" rpy="0.000 0.000 0.000" />
+            </collision>
+            <inertial>
+                <mass value="2.161679" />
+                <origin xyz="0.014568 -0.016319 0.019397" rpy="0 0 0" />
+                <inertia ixx="0.007515" ixy="-0.001184" ixz="-0.000026"
+                        iyy="0.003859" iyz="0.000191"
+                        izz="0.010255" />
             </inertial>
         </link>
@@ -41,12 +41,12 @@
             <visual>
                 <geometry>
-                <mesh filename="package://a6x_description/meshes/visual/shoulder_link.STL" />
-                </geometry>
-                <origin xyz="0.000 0.000 0.000" rpy="0.000 0.000 0.000" />
-                <material name="grey" />
-            </visual>
-            <collision>
-                <geometry>
-                <mesh filename="package://a6x_description/meshes/visual/shoulder_link.STL" />
+                    <mesh filename="package://a6x_description/meshes/visual/shoulder_link.STL" />
+                </geometry>
+                <origin xyz="0.000 0.000 0.000" rpy="0.000 0.000 0.000" />
+                <material name="grey" />
+            </visual>
+            <collision>
+                <geometry>
+                    <mesh filename="package://a6x_description/meshes/visual/shoulder_link.STL" />
                 </geometry>
                 <origin xyz="0.000 0.000 0.000" rpy="0.000 0.000 0.000" />
@@ -70,12 +70,12 @@
             <visual>
                 <geometry>
-                <mesh filename="package://a6x_description/meshes/visual/arm_link.STL" />
-                </geometry>
-                <origin xyz="0.000 0.000 0.000" rpy="0.000 0.000 0.000" />
-                <material name="grey" />
-            </visual>
-            <collision>
-                <geometry>
-                <mesh filename="package://a6x_description/meshes/visual/arm_link.STL" />
+                    <mesh filename="package://a6x_description/meshes/visual/arm_link.STL" />
+                </geometry>
+                <origin xyz="0.000 0.000 0.000" rpy="0.000 0.000 0.000" />
+                <material name="grey" />
+            </visual>
+            <collision>
+                <geometry>
+                    <mesh filename="package://a6x_description/meshes/visual/arm_link.STL" />
                 </geometry>
                 <origin xyz="0.000 0.000 0.000" rpy="0.000 0.000 0.000" />
@@ -99,12 +99,12 @@
             <visual>
                 <geometry>
-                <mesh filename="package://a6x_description/meshes/visual/forearm_link.STL" />
-                </geometry>
-                <origin xyz="0.000 0.000 0.000" rpy="0.000 0.000 0.000" />
-                <material name="grey" />
-            </visual>
-            <collision>
-                <geometry>
-                <mesh filename="package://a6x_description/meshes/visual/forearm_link.STL" />
+                    <mesh filename="package://a6x_description/meshes/visual/forearm_link.STL" />
+                </geometry>
+                <origin xyz="0.000 0.000 0.000" rpy="0.000 0.000 0.000" />
+                <material name="grey" />
+            </visual>
+            <collision>
+                <geometry>
+                    <mesh filename="package://a6x_description/meshes/visual/forearm_link.STL" />
                 </geometry>
                 <origin xyz="0.000 0.000 0.000" rpy="0.000 0.000 0.000" />
@@ -128,12 +128,12 @@
             <visual>
                 <geometry>
-                <mesh filename="package://a6x_description/meshes/visual/lower_wrist_link.STL" />
-                </geometry>
-                <origin xyz="0.000 0.000 0.000" rpy="0.000 0.000 0.000" />
-                <material name="grey" />
-            </visual>
-            <collision>
-                <geometry>
-                <mesh filename="package://a6x_description/meshes/visual/lower_wrist_link.STL" />
+                    <mesh filename="package://a6x_description/meshes/visual/lower_wrist_link.STL" />
+                </geometry>
+                <origin xyz="0.000 0.000 0.000" rpy="0.000 0.000 0.000" />
+                <material name="grey" />
+            </visual>
+            <collision>
+                <geometry>
+                    <mesh filename="package://a6x_description/meshes/visual/lower_wrist_link.STL" />
                 </geometry>
                 <origin xyz="0.000 0.000 0.000" rpy="0.000 0.000 0.000" />
@@ -157,21 +157,21 @@
             <visual>
                 <geometry>
-                <mesh filename="package://a6x_description/meshes/visual/upper_wrist_link.STL" />
-                </geometry>
-                <origin xyz="0.000 0.000 0.000" rpy="0.000 0.000 0.000" />
-                <material name="grey" />
-            </visual>
-            <collision>
-                <geometry>
-                <mesh filename="package://a6x_description/meshes/visual/upper_wrist_link.STL" />
-                </geometry>
-                <origin xyz="0.000 0.000 0.000" rpy="0.000 0.000 0.000" />
-            </collision>
-            <inertial>
-                <mass value="0.279057" />
-                <origin xyz="-0.001436 0.028250 0.000000" rpy="0 0 0" />
-                <inertia ixx="0.000143" ixy="0.000005" ixz="0.000000"
-                        iyy="0.000087" iyz="0.000000"
-                        izz="0.000135" />
+                    <mesh filename="package://a6x_description/meshes/visual/upper_wrist_link.STL" />
+                </geometry>
+                <origin xyz="0.000 0.000 0.000" rpy="0.000 0.000 0.000" />
+                <material name="grey" />
+            </visual>
+            <collision>
+                <geometry>
+                    <mesh filename="package://a6x_description/meshes/visual/upper_wrist_link.STL" />
+                </geometry>
+                <origin xyz="0.000 0.000 0.000" rpy="0.000 0.000 0.000" />
+            </collision>
+            <inertial>
+                <mass value="0.313268" />
+                <origin xyz="-0.000382 0.031134 0.000487" rpy="0 0 0" />
+                <inertia ixx="0.000165" ixy="-0.000002" ixz="0.000000"
+                        iyy="0.000124" iyz="0.000001"
+                        izz="0.000182" />
             </inertial>
         </link>
@@ -179,28 +179,28 @@
             <parent link="upper_wrist_link" />
             <child link="palm_link" />
-            <origin xyz="0.019 0.055 0.000" rpy="0 0 0" />
+            <origin xyz="0.022 0.044 0.001" rpy="0 0 0" />
             <axis xyz="1 0 0" />
-            <limit lower="0" upper="6.28" effort="10" velocity="1.0" />
+            <limit lower="-3.14" upper="3.14" effort="10" velocity="1.0" />
         </joint>
         <link name="palm_link">
             <visual>
                 <geometry>
-                <mesh filename="package://a6x_description/meshes/visual/palm_link.STL" />
-                </geometry>
-                <origin xyz="0.000 0.000 0.000" rpy="0.000 0.000 0.000" />
-                <material name="grey" />
-            </visual>
-            <collision>
-                <geometry>
-                <mesh filename="package://a6x_description/meshes/visual/palm_link.STL" />
-                </geometry>
-                <origin xyz="0.000 0.000 0.000" rpy="0.000 0.000 0.000" />
-            </collision>
-            <inertial>
-                <mass value="0.216056" />
-                <origin xyz="0.026410 0.000000 -0.008366" rpy="0 0 0" />
-                <inertia ixx="0.000145" ixy="0.000000" ixz="0.000007"
-                        iyy="0.000080" iyz="0.000000"
-                        izz="0.000126" />
+                    <mesh filename="package://a6x_description/meshes/visual/palm_link.STL" />
+                </geometry>
+                <origin xyz="0.000 0.000 0.000" rpy="0.000 0.000 0.000" />
+                <material name="grey" />
+            </visual>
+            <collision>
+                <geometry>
+                    <mesh filename="package://a6x_description/meshes/visual/palm_link.STL" />
+                </geometry>
+                <origin xyz="0.000 0.000 0.000" rpy="0.000 0.000 0.000" />
+            </collision>
+            <inertial>
+                <mass value="0.342542" />
+                <origin xyz="0.040329 0.000003 0.000000" rpy="0 0 0" />
+                <inertia ixx="0.000231" ixy="0.000000" ixz="0.000000"
+                        iyy="0.000170" iyz="-0.000002"
+                        izz="0.000299" />
             </inertial>
         </link>
@@ -208,5 +208,5 @@
             <parent link="palm_link" />
             <child link="left_finger_link" />
-            <origin xyz="0.038 -0.040 0.016" rpy="0 0 0" />
+            <origin xyz="0.057 -0.048 0.016" rpy="0 0 0" />
             <axis xyz="0 -1 0" />
             <limit lower="-0.010" upper="0.019" effort="1" velocity="4.8" />
@@ -216,19 +216,19 @@
             <parent link="palm_link" />
             <child link="right_finger_link" />
-            <origin xyz="0.038 0.040 0.016" rpy="0 0 0" />
+            <origin xyz="0.057 0.048 0.016" rpy="0 0 0" />
             <axis xyz="0 -1 0" />
-            <limit lower="-0.010" upper="0.019" effort="1" velocity="4.8" />
+            <limit lower="-0.019" upper="0.010" effort="1" velocity="4.8" />
         </joint>
         <link name="left_finger_link">
             <visual>
                 <geometry>
-                <mesh filename="package://a6x_description/meshes/visual/left_finger_link.STL" />
-                </geometry>
-                <origin xyz="0.000 0.000 0.000" rpy="0.000 0.000 0.000" />
-                <material name="grey" />
-            </visual>
-            <collision>
-                <geometry>
-                <mesh filename="package://a6x_description/meshes/visual/left_finger_link.STL" />
+                    <mesh filename="package://a6x_description/meshes/visual/left_finger_link.STL" />
+                </geometry>
+                <origin xyz="0.000 0.000 0.000" rpy="0.000 0.000 0.000" />
+                <material name="grey" />
+            </visual>
+            <collision>
+                <geometry>
+                    <mesh filename="package://a6x_description/meshes/visual/left_finger_link.STL" />
                 </geometry>
                 <origin xyz="0.000 0.000 0.000" rpy="0.000 0.000 0.000" />
@@ -245,16 +245,16 @@
             <visual>
                 <geometry>
-                <mesh filename="package://a6x_description/meshes/visual/right_finger_link.STL" />
-                </geometry>
-                <origin xyz="0.000 0.000 0.000" rpy="0.000 0.000 0.000" />
-                <material name="grey" />
-            </visual>
-            <collision>
-                <geometry>
-                <mesh filename="package://a6x_description/meshes/visual/right_finger_link.STL" />
-                </geometry>
-                <origin xyz="0.000 0.000 0.000" rpy="0.000 0.000 0.000" />
-            </collision>
-                    <inertial>
+                    <mesh filename="package://a6x_description/meshes/visual/right_finger_link.STL" />
+                </geometry>
+                <origin xyz="0.000 0.000 0.000" rpy="0.000 0.000 0.000" />
+                <material name="grey" />
+            </visual>
+            <collision>
+                <geometry>
+                    <mesh filename="package://a6x_description/meshes/visual/right_finger_link.STL" />
+                </geometry>
+                <origin xyz="0.000 0.000 0.000" rpy="0.000 0.000 0.000" />
+            </collision>
+                <inertial>
                 <mass value="0.111661" />
                 <origin xyz="0.036898 -0.012549 -0.016201" rpy="0 0 0" />
