Commit message: update new lower and upper limit for joint urdf

File: a6x_description/urdf/a6x.urdf (robot description, URDF)
Before this commit: robot arm, 9 links, 8 joints
Joints:
- joint forearm_roll_joint: limit lower=-1.5 upper=1.5 effort=10 velocity=1.0 -> lower=-5.393 upper=0.205 effort=10 velocity=1.0
- joint lower_wrist_roll_joint: limit lower=-1.5 upper=1.5 effort=10 velocity=1.0 -> lower=-3.14 upper=3.14 effort=10 velocity=1.0
- joint palm_roll_joint: limit lower=-1.5 upper=1.5 effort=10 velocity=1.0 -> lower=-3.14 upper=3.14 effort=10 velocity=1.0
- joint upper_wrist_pitch_joint: limit lower=-1.5 upper=1.5 effort=10 velocity=1.0 -> lower=-1.57 upper=1.57 effort=10 velocity=1.0

Commit message: new hardware interface for dynamixel and robstride

File: a6x_description/urdf/a6x.urdf (robot description, URDF)
Before this commit: robot arm, 9 links, 8 joints
Links:
- link arm_link: mass 1.783675 -> 1.691838
- link base_link: mass 2.020908 -> 2.052381
- link forearm_link: mass 1.581202 -> 1.652648
- link shoulder_link: mass 0.367611 -> 0.453182
- link upper_wrist: mass 0.284324 -> 0.279057
Joints:
- joint arm_roll_joint: origin xyz=-0.037 0.000 0.060 rpy=0 0 0 -> xyz=-0.039 0.000 0.070 rpy=0 0 0
- joint forearm_roll_joint: limit lower=-5.393 upper=0.205 effort=10 velocity=1.0 -> lower=-5.350 upper=0.205 effort=10 velocity=1.0; origin xyz=-0.003 -0.278 0.114 rpy=0 0 0 -> xyz=0.000 -0.283 0.100 rpy=0 0 0
- joint left_finger_prismatic_joint: axis 0 1 0 -> 0 -1 0; limit lower=-0.013 upper=0.013 effort=100.0 velocity=0.05 -> lower=-0.010 upper=0.019 effort=1 velocity=4.8
- joint lower_wrist_roll_joint: origin xyz=0.059 0.134 -0.188 rpy=0 0 0 -> xyz=0.059 0.139 -0.185 rpy=0 0 0
- joint right_finger_prismatic_joint: axis 0 1 0 -> 0 -1 0; limit lower=-0.013 upper=0.013 effort=100.0 velocity=0.05 -> lower=-0.019 upper=0.010 effort=1 velocity=4.8

File: a6x_description/urdf/a6x_macro.urdf.xacro (robot description, xacro)
@@ -5,6 +5,6 @@
 <!-- =================================================================================== -->
 <robot xmlns:xacro="http://ros.org/wiki/xacro">
-    <material name="aquablue">
-        <color rgba="0.00784313725490196 0.8470588235294118 0.9137254901960784 1.0" />
+    <material name="grey">
+        <color rgba="0.64 0.64 0.64 1.0" />
     </material>
     <xacro:macro name="a6x_robot">
@@ -15,5 +15,5 @@
                 </geometry>
                 <origin xyz="0.000 0.000 0.000" rpy="0.000 0.000 0.000" />
-                <material name="aquablue" />
+                <material name="grey" />
             </visual>
             <collision>
@@ -24,9 +24,9 @@
             </collision>
             <inertial>
-                <mass value="2.020908" />
-                <origin xyz="0.010364 -0.013298 0.019441" rpy="0 0 0" />
-                <inertia ixx="0.007042" ixy="-0.000717" ixz="-0.000018"
-                        iyy="0.003221" iyz="0.000166"
-                        izz="0.009183" />
+                <mass value="2.052381" />
+                <origin xyz="0.010773 -0.013141 0.019508" rpy="0 0 0" />
+                <inertia ixx="0.007060" ixy="-0.000705" ixz="-0.000013"
+                        iyy="0.003238" iyz="0.000167"
+                        izz="0.009216" />
             </inertial>
         </link>
@@ -44,5 +44,5 @@
                 </geometry>
                 <origin xyz="0.000 0.000 0.000" rpy="0.000 0.000 0.000" />
-                <material name="aquablue" />
+                <material name="grey" />
             </visual>
             <collision>
@@ -53,9 +53,9 @@
             </collision>
             <inertial>
-                <mass value="0.367611" />
-                <origin xyz="0.000000 -0.000082 0.019648" rpy="0 0 0" />
-                <inertia ixx="0.000415" ixy="0.000000" ixz="0.000000"
-                        iyy="0.000537" iyz="-0.000001"
-                        izz="0.000645" />
+                <mass value="0.453182" />
+                <origin xyz="-0.012231 0.000430 0.037054" rpy="0 0 0" />
+                <inertia ixx="0.000959" ixy="0.000002" ixz="-0.000103"
+                        iyy="0.000618" iyz="-0.000004"
+                        izz="0.000763" />
             </inertial>
         </link>
@@ -63,6 +63,6 @@
             <parent link="shoulder_link" />
             <child link="arm_link" />
-            <origin xyz="-0.037 0.000 0.060" rpy="0 0 0" />
-            <axis xyz="1 0 0" />
+            <origin xyz="-0.039 0.000 0.070" rpy="0 0 0" />
+            <axis xyz="-1 0 0" />
             <limit lower="-2.967" upper="0.785" effort="10" velocity="1.0" />
         </joint>
@@ -73,5 +73,5 @@
                 </geometry>
                 <origin xyz="0.000 0.000 0.000" rpy="0.000 0.000 0.000" />
-                <material name="aquablue" />
+                <material name="grey" />
             </visual>
             <collision>
@@ -82,9 +82,9 @@
             </collision>
             <inertial>
-                <mass value="1.783675" />
-                <origin xyz="0.035891 -0.069538 0.028493" rpy="0 0 0" />
-                <inertia ixx="0.027167" ixy="-0.000287" ixz="0.000116"
-                        iyy="0.007550" iyz="-0.009088"
-                        izz="0.026001" />
+                <mass value="1.691838" />
+                <origin xyz="0.031472 -0.101109 0.035700" rpy="0 0 0" />
+                <inertia ixx="0.024919" ixy="0.000300" ixz="-0.000105"
+                        iyy="0.006756" iyz="-0.007400"
+                        izz="0.024952" />
             </inertial>
         </link>
@@ -92,7 +92,7 @@
             <parent link="arm_link" />
             <child link="forearm_link" />
-            <origin xyz="-0.003 -0.278 0.114" rpy="0 0 0" />
+            <origin xyz="0.000 -0.283 0.100" rpy="0 0 0" />
             <axis xyz="-1 0 0" />
-            <limit lower="-5.393" upper="0.205" effort="10" velocity="1.0" />
+            <limit lower="-5.350" upper="0.205" effort="10" velocity="1.0" />
         </joint>
         <link name="forearm_link">
@@ -102,5 +102,5 @@
                 </geometry>
                 <origin xyz="0.000 0.000 0.000" rpy="0.000 0.000 0.000" />
-                <material name="aquablue" />
+                <material name="grey" />
             </visual>
             <collision>
@@ -111,9 +111,9 @@
             </collision>
             <inertial>
-                <mass value="1.581202" />
-                <origin xyz="0.037295 0.060924 -0.085845" rpy="0 0 0" />
-                <inertia ixx="0.018638" ixy="0.000243" ixz="-0.000341"
-                        iyy="0.012327" iyz="-0.007973"
-                        izz="0.006798" />
+                <mass value="1.652648" />
+                <origin xyz="0.037370 0.063424 -0.084543" rpy="0 0 0" />
+                <inertia ixx="0.018666" ixy="0.000252" ixz="-0.000337"
+                        iyy="0.011953" iyz="-0.008070"
+                        izz="0.007223" />
             </inertial>
         </link>
@@ -121,5 +121,5 @@
             <parent link="forearm_link" />
             <child link="lower_wrist" />
-            <origin xyz="0.059 0.134 -0.188" rpy="0 0 0" />
+            <origin xyz="0.059 0.139 -0.185" rpy="0 0 0" />
             <axis xyz="1 0 0" />
             <limit lower="-3.14" upper="3.14" effort="10" velocity="1.0" />
@@ -131,5 +131,5 @@
                 </geometry>
                 <origin xyz="0.000 0.000 0.000" rpy="0.000 0.000 0.000" />
-                <material name="aquablue" />
+                <material name="grey" />
             </visual>
             <collision>
@@ -141,5 +141,5 @@
             <inertial>
                 <mass value="0.628723" />
-                <origin xyz="0.052187 0.000876 0.000348" rpy="0 0 0" />
+                <origin xyz="0.052187 0.000889 0.000348" rpy="0 0 0" />
                 <inertia ixx="0.000438" ixy="-0.000003" ixz="0.000002"
                         iyy="0.000865" iyz="-0.000001"
@@ -160,5 +160,5 @@
                 </geometry>
                 <origin xyz="0.000 0.000 0.000" rpy="0.000 0.000 0.000" />
-                <material name="aquablue" />
+                <material name="grey" />
             </visual>
             <collision>
@@ -169,9 +169,97 @@
             </collision>
             <inertial>
-                <mass value="0.284324" />
-                <origin xyz="-0.000993 0.027842 0.000000" rpy="0 0 0" />
-                <inertia ixx="0.000146" ixy="0.000003" ixz="0.000000"
-                        iyy="0.000090" iyz="0.000000"
-                        izz="0.000141" />
+                <mass value="0.279057" />
+                <origin xyz="-0.001436 0.028250 0.000000" rpy="0 0 0" />
+                <inertia ixx="0.000143" ixy="0.000005" ixz="0.000000"
+                        iyy="0.000087" iyz="0.000000"
+                        izz="0.000135" />
+            </inertial>
+        </link>
+        <joint name="palm_roll_joint" type="revolute">
+            <parent link="upper_wrist" />
+            <child link="palm_link" />
+            <origin xyz="0.019 0.055 0.000" rpy="0 0 0" />
+            <axis xyz="1 0 0" />
+            <limit lower="0" upper="6.28" effort="10" velocity="1.0" />
+        </joint>
+        <link name="palm_link">
+            <visual>
+                <geometry>
+                <mesh filename="package://a6x_description/meshes/visual/palm_link.STL" />
+                </geometry>
+                <origin xyz="0.000 0.000 0.000" rpy="0.000 0.000 0.000" />
+                <material name="grey" />
+            </visual>
+            <collision>
+                <geometry>
+                <mesh filename="package://a6x_description/meshes/visual/palm_link.STL" />
+                </geometry>
+                <origin xyz="0.000 0.000 0.000" rpy="0.000 0.000 0.000" />
+            </collision>
+            <inertial>
+                <mass value="0.216056" />
+                <origin xyz="0.026410 0.000000 -0.008366" rpy="0 0 0" />
+                <inertia ixx="0.000145" ixy="0.000000" ixz="0.000007"
+                        iyy="0.000080" iyz="0.000000"
+                        izz="0.000126" />
+            </inertial>
+        </link>
+        <joint name="left_finger_prismatic_joint" type="prismatic">
+            <parent link="palm_link" />
+            <child link="left_finger_link" />
+            <origin xyz="0.038 -0.040 0.016" rpy="0 0 0" />
+            <axis xyz="0 -1 0" />
+            <limit lower="-0.010" upper="0.019" effort="1" velocity="4.8" />
+        </joint>
+        <joint name="right_finger_prismatic_joint" type="prismatic">
+            <mimic joint="left_finger_prismatic_joint" multiplier="-1" offset="0" />
+            <parent link="palm_link" />
+            <child link="right_finger_link" />
+            <origin xyz="0.038 0.040 0.016" rpy="0 0 0" />
+            <axis xyz="0 -1 0" />
+            <limit lower="-0.019" upper="0.010" effort="1" velocity="4.8" />
+        </joint>
+        <link name="left_finger_link">
+            <visual>
+                <geometry>
+                <mesh filename="package://a6x_description/meshes/visual/left_finger_link.STL" />
+                </geometry>
+                <origin xyz="0.000 0.000 0.000" rpy="0.000 0.000 0.000" />
+                <material name="grey" />
+            </visual>
+            <collision>
+                <geometry>
+                <mesh filename="package://a6x_description/meshes/visual/left_finger_link.STL" />
+                </geometry>
+                <origin xyz="0.000 0.000 0.000" rpy="0.000 0.000 0.000" />
+            </collision>
+            <inertial>
+                <mass value="0.111661" />
+                <origin xyz="0.036901 0.012552 -0.016199" rpy="0 0 0" />
+                <inertia ixx="0.000028" ixy="0.000012" ixz="0.000000"
+                        iyy="0.000075" iyz="0.000000"
+                        izz="0.000065" />
+            </inertial>
+        </link>
+        <link name="right_finger_link">
+            <visual>
+                <geometry>
+                <mesh filename="package://a6x_description/meshes/visual/right_finger_link.STL" />
+                </geometry>
+                <origin xyz="0.000 0.000 0.000" rpy="0.000 0.000 0.000" />
+                <material name="grey" />
+            </visual>
+            <collision>
+                <geometry>
+                <mesh filename="package://a6x_description/meshes/visual/right_finger_link.STL" />
+                </geometry>
+                <origin xyz="0.000 0.000 0.000" rpy="0.000 0.000 0.000" />
+            </collision>
+                    <inertial>
+                <mass value="0.111661" />
+                <origin xyz="0.036898 -0.012549 -0.016201" rpy="0 0 0" />
+                <inertia ixx="0.000028" ixy="-0.000012" ixz="0.000000"
+                        iyy="0.000075" iyz="0.000000"
+                        izz="0.000065" />
             </inertial>
         </link>

File: a6x_ros2_control/description/urdf/a6x.urdf.xacro (robot description, xacro)
@@ -2,13 +2,22 @@
 <robot name="a6x_robot" xmlns:xacro="http://www.ros.org/wiki/xacro">
     <xacro:property name="serial_port" default="/dev/ttyUSB0" />
+    <xacro:property name="serial_port1" default="/dev/ttyUSB1" />
+    <xacro:property name="canbus" default="can0" />
     <xacro:include filename="$(find a6x_description)/urdf/a6x_macro.urdf.xacro" />
     <xacro:include filename="$(find unitree_hardware)/description/ros2_control/unitree_motor.ros2_control.urdf.xacro" />
+    <xacro:include filename="$(find cybergear_control)/description/ros2_control/robstride.ros2_control.urdf.xacro"/>
+    <xacro:include filename="$(find dynamixel_hardware_interface)/description/ros2_control/dynamixel_motor.ros2_control.xacro"/>
     <!-- expand the robot macro to include links and joints defined in a6x_macro -->
     <xacro:a6x_robot />
     <!-- ros2_control hardware systems for motors -->
-    <xacro:unitree_ros2_control name="ShoulderYaw" serial_device="${serial_port}" device_id="0" joint_name="shoulder_yaw_joint" />
-    <xacro:unitree_ros2_control name="ArmRoll" serial_device="${serial_port}" device_id="1" joint_name="arm_roll_joint" />
+    <xacro:unitree_ros2_control name="ShoulderYaw" serial_device="${serial_port}" device_id="1" joint_name="shoulder_yaw_joint" />
+    <xacro:robstride_ros2_control name="ArmRoll" canbus="${canbus}" device_id="2" joint_name="arm_roll_joint"/>
     <xacro:unitree_ros2_control name="ForearmRoll" serial_device="${serial_port}" device_id="3" joint_name="forearm_roll_joint" />
     <xacro:unitree_ros2_control name="LowerWristRoll" serial_device="${serial_port}" device_id="4" joint_name="lower_wrist_roll_joint" />
     <xacro:unitree_ros2_control name="UpperWristPitch" serial_device="${serial_port}" device_id="5" joint_name="upper_wrist_pitch_joint" />
+    <xacro:dynamixel_ros2_control name="PalmRoll" serial_device="${serial_port1}" device_id="6" joint_name="palm_roll_joint" />
+    <xacro:dynamixel_ros2_control name="LeftFingerPrismatic" serial_device="${serial_port1}" device_id="7" joint_name="left_finger_prismatic_joint"
+                                  use_prismatic="1"
+                                  revolute_max="-1.52" revolute_min="0.92"
+                                  prismatic_max="0.019" prismatic_min="-0.01" />
 </robot>

Commit message: update new version moveit and fix dynamixel finger state_interfaces error

File: a6x_description/urdf/a6x.urdf (robot description, URDF)
Before this commit: robot arm, 9 links, 8 joints
Joints:
- joint arm_roll_joint: axis 1 0 0 -> -1 0 0; limit lower=-2.967 upper=0.785 effort=10 velocity=1.0 -> lower=-0.785 upper=2.967 effort=10 velocity=1.0
- joint forearm_roll_joint: axis 1 0 0 -> -1 0 0; limit lower=-5.350 upper=0.205 effort=10 velocity=1.0 -> lower=-0.205 upper=5.350 effort=10 velocity=1.0

File: a6x_description/urdf/a6x_macro.urdf.xacro (robot description, xacro)
@@ -65,5 +65,5 @@
             <origin xyz="-0.039 0.000 0.070" rpy="0 0 0" />
             <axis xyz="-1 0 0" />
-            <limit lower="-2.967" upper="0.785" effort="10" velocity="1.0" />
+            <limit lower="-0.785" upper="2.967" effort="10" velocity="1.0" />
         </joint>
         <link name="arm_link">
@@ -94,5 +94,5 @@
             <origin xyz="0.000 -0.283 0.100" rpy="0 0 0" />
             <axis xyz="-1 0 0" />
-            <limit lower="-5.350" upper="0.205" effort="10" velocity="1.0" />
+            <limit lower="-0.205" upper="5.350" effort="10" velocity="1.0" />
         </joint>
         <link name="forearm_link">
@@ -218,5 +218,5 @@
             <origin xyz="0.038 0.040 0.016" rpy="0 0 0" />
             <axis xyz="0 -1 0" />
-            <limit lower="-0.019" upper="0.010" effort="1" velocity="4.8" />
+            <limit lower="-0.010" upper="0.019" effort="1" velocity="4.8" />
         </joint>
         <link name="left_finger_link">

File: a6x_moveit_config/config/a6x_robot.ros2_control.xacro (robot description, xacro)
@@ -1,5 +1,5 @@
 <?xml version="1.0"?>
 <robot xmlns:xacro="http://www.ros.org/wiki/xacro">
-    <xacro:macro name="arm_ros2_control" params="name initial_positions_file">
+    <xacro:macro name="a6x_robot_ros2_control" params="name initial_positions_file">
         <xacro:property name="initial_positions" value="${load_yaml(initial_positions_file)['initial_positions']}"/>
         <ros2_control name="${name}" type="system">

File: a6x_ros2_control/description/urdf/a6x.urdf.xacro (robot description, xacro)
@@ -19,5 +19,5 @@
     <xacro:dynamixel_ros2_control name="LeftFingerPrismatic" serial_device="${serial_port1}" device_id="7" joint_name="left_finger_prismatic_joint"
                                   use_prismatic="1"
-                                  revolute_max="-1.52" revolute_min="0.92"
-                                  prismatic_max="0.019" prismatic_min="-0.01" />
+                                  revolute_max="0.0" revolute_min="-2.5"
+                                  prismatic_max="0.019" prismatic_min="-0.013" />
 </robot>

File: cybergear_hardware/cybergear_servo_description/urdf/cybergear_servo.xacro (robot description, xacro)
@@ -20,5 +20,5 @@
         <origin rpy="0 0 0" xyz="0 0 0.008"/>
         <geometry>
-          <cylinder length="0.035" radius="0.042"/>
+          <cylinder length="0.035" radius="0.042"/>>
         </geometry>
       </collision>
@@ -33,5 +33,5 @@
       <origin rpy="0 0 0" xyz="0 0 0.028"/>
       <parent link="${name}_cybergear_link"/>
-      <child link="${name}_cybergear_table_link"/>
+      <child link="${name}_cybergear_table_link"/>>
       <axis xyz="0 0 1"/>
       <limit effort="12" velocity="30" lower="-12.565" upper="12.565"/>
