Commit message: adding end_effector and moveit config

File: a6x_description/urdf/a6x.urdf (robot description, URDF)
Before this commit: robot a6x_robot, 9 links, 8 joints
Links:
- removed link lower_wrist
- removed link upper_wrist
- added link camera_link, mass 0.028176; collision mesh filename=package://a6x_description/meshes/visual/camera_link.STL; visual mesh filename=package://a6x_description/meshes/visual/camera_link.STL
- added link end_effector_link
- added link lower_wrist_link, mass 0.628723; collision mesh filename=package://a6x_description/meshes/visual/lower_wrist_link.STL; visual mesh filename=package://a6x_description/meshes/visual/lower_wrist_link.STL
- added link upper_wrist_link, mass 0.279057; collision mesh filename=package://a6x_description/meshes/visual/upper_wrist_link.STL; visual mesh filename=package://a6x_description/meshes/visual/upper_wrist_link.STL
Joints:
- added joint camera_fixed_joint: type fixed, parent upper_wrist_link, child camera_link, origin xyz=-0.013 0.041 0.014 rpy=0 0 0
- added joint end_effector_fixed_joint: type fixed, parent palm_link, child end_effector_link, origin xyz=0.1 0.000 0.000 rpy=0 0 0
- joint lower_wrist_roll_joint: child lower_wrist -> lower_wrist_link
- joint palm_roll_joint: parent upper_wrist -> upper_wrist_link
- joint upper_wrist_pitch_joint: child upper_wrist -> upper_wrist_link; parent lower_wrist -> lower_wrist_link

File: a6x_description/urdf/a6x_macro.urdf.xacro (robot description, xacro)
@@ -120,10 +120,10 @@
         <joint name="lower_wrist_roll_joint" type="revolute">
             <parent link="forearm_link" />
-            <child link="lower_wrist" />
+            <child link="lower_wrist_link" />
             <origin xyz="0.059 0.139 -0.185" rpy="0 0 0" />
             <axis xyz="1 0 0" />
             <limit lower="-3.14" upper="3.14" effort="10" velocity="1.0" />
         </joint>
-        <link name="lower_wrist">
+        <link name="lower_wrist_link">
             <visual>
                 <geometry>
@@ -148,11 +148,11 @@
         </link>
         <joint name="upper_wrist_pitch_joint" type="revolute">
-            <parent link="lower_wrist" />
-            <child link="upper_wrist" />
+            <parent link="lower_wrist_link" />
+            <child link="upper_wrist_link" />
             <origin xyz="0.060 0.020 0.000" rpy="0 0 0" />
             <axis xyz="0 1 0" />
             <limit lower="-1.57" upper="1.57" effort="10" velocity="1.0" />
         </joint>
-        <link name="upper_wrist">
+        <link name="upper_wrist_link">
             <visual>
                 <geometry>
@@ -176,6 +176,33 @@
             </inertial>
         </link>
+    <joint name="camera_fixed_joint" type="fixed">
+        <parent link="upper_wrist_link" />
+        <child link="camera_link" />
+        <origin xyz="-0.013 0.041 0.014" rpy="0 0 0" />
+    </joint>
+    <link name="camera_link">
+        <visual>
+            <geometry>
+               <mesh filename="package://a6x_description/meshes/visual/camera_link.STL" />
+            </geometry>
+            <origin xyz="0.000 0.000 0.000" rpy="0.000 0.000 0.000" />
+            <material name="grey" />
+        </visual>
+        <collision>
+            <geometry>
+               <mesh filename="package://a6x_description/meshes/visual/camera_link.STL" />
+        </geometry>
+            <origin xyz="0.000 0.000 0.000" rpy="0.000 0.000 0.000" />
+        </collision>
+        <inertial>
+            <mass value="0.028176" />
+            <origin xyz="0.000530 -0.008677 0.020667" rpy="0 0 0" />
+            <inertia ixx="0.000005" ixy="0.000000" ixz="0.000000"
+                     iyy="0.000002" iyz="-0.000001"
+                     izz="0.000004" />
+        </inertial>
+    </link>
         <joint name="palm_roll_joint" type="revolute">
-            <parent link="upper_wrist" />
+            <parent link="upper_wrist_link" />
             <child link="palm_link" />
             <origin xyz="0.019 0.055 0.000" rpy="0 0 0" />
@@ -264,4 +291,10 @@
             </inertial>
         </link>
+        <joint name="end_effector_fixed_joint" type="fixed">
+            <parent link="palm_link" />
+            <child link="end_effector_link" />
+            <origin xyz="0.1 0.000 0.000" rpy="0 0 0" />
+        </joint>
+        <link name="end_effector_link" />
     </xacro:macro>
 </robot>

File: unitree_hardware/description/ros2_control/unitree_motor.ros2_control.urdf.xacro (robot description, xacro)
@@ -10,6 +10,6 @@
                 <param name="id">${device_id}</param>
                 <param name="motor_type">GO-M8010-6</param>
-                <param name="pos_gain">30.0</param>
-                <param name="vel_gain">1.0</param>
+                <param name="pos_gain">230.0</param>
+                <param name="vel_gain">5.0</param>
                 <param name="temperature_limit">80.</param>
                 <command_interface name="position" />

Commit message: urdf camera_link removed & update launch file to match moveit

File: a6x_description/urdf/a6x.urdf (robot description, URDF)
Before this commit: robot a6x_robot, 11 links, 10 joints
Links:
- removed link camera_link
Joints:
- removed joint camera_fixed_joint

File: a6x_description/urdf/a6x_macro.urdf.xacro (robot description, xacro)
@@ -176,31 +176,4 @@
             </inertial>
         </link>
-    <joint name="camera_fixed_joint" type="fixed">
-        <parent link="upper_wrist_link" />
-        <child link="camera_link" />
-        <origin xyz="-0.013 0.041 0.014" rpy="0 0 0" />
-    </joint>
-    <link name="camera_link">
-        <visual>
-            <geometry>
-               <mesh filename="package://a6x_description/meshes/visual/camera_link.STL" />
-            </geometry>
-            <origin xyz="0.000 0.000 0.000" rpy="0.000 0.000 0.000" />
-            <material name="grey" />
-        </visual>
-        <collision>
-            <geometry>
-               <mesh filename="package://a6x_description/meshes/visual/camera_link.STL" />
-        </geometry>
-            <origin xyz="0.000 0.000 0.000" rpy="0.000 0.000 0.000" />
-        </collision>
-        <inertial>
-            <mass value="0.028176" />
-            <origin xyz="0.000530 -0.008677 0.020667" rpy="0 0 0" />
-            <inertia ixx="0.000005" ixy="0.000000" ixz="0.000000"
-                     iyy="0.000002" iyz="-0.000001"
-                     izz="0.000004" />
-        </inertial>
-    </link>
         <joint name="palm_roll_joint" type="revolute">
             <parent link="upper_wrist_link" />
