Commit message: Update new Robot's arm, i defined new base_link, upper_wrist_link, and palm_link's mass and inertia, and also update the urdf file.

File: a6x_description/urdf/a6x.urdf (robot description, URDF)
Before this commit: robot a6x_robot, 10 links, 9 joints
Links:
- link base_link: mass 2.052381 -> 2.161679
- link palm_link: mass 0.216056 -> 0.342542
- link upper_wrist_link: mass 0.279057 -> 0.313268
Joints:
- joint left_finger_prismatic_joint: origin xyz=0.038 -0.040 0.016 rpy=0 0 0 -> xyz=0.057 -0.048 0.016 rpy=0 0 0
- joint palm_roll_joint: origin xyz=0.019 0.055 0.000 rpy=0 0 0 -> xyz=0.022 0.044 0.001 rpy=0 0 0
- joint right_finger_prismatic_joint: origin xyz=0.038 0.040 0.016 rpy=0 0 0 -> xyz=0.057 0.048 0.016 rpy=0 0 0
